Commit message: side view too low

File: src/ur20_sim/urdf/ur20_parked.urdf.xacro (robot description, xacro)
@@ -7,3 +7,28 @@
   <xacro:arg name="initial_positions_file" default="$(find ur20_sim)/config/initial_positions.yaml"/>
   <xacro:include filename="$(find ur_description)/urdf/ur.urdf.xacro"/>
+  <!-- Camera sticking 22 cm out of the flange along tool z. Modeled as a
+       cylinder so MoveIt collision-checks it against the room. Starts 1 cm
+       past the flange to avoid false self-collision with wrist_3. -->
+  <link name="camera">
+    <visual>
+      <origin xyz="0 0 0.115" rpy="0 0 0"/>
+      <geometry>
+        <cylinder radius="0.03" length="0.21"/>
+      </geometry>
+      <material name="camera_grey">
+        <color rgba="0.3 0.3 0.3 1.0"/>
+      </material>
+    </visual>
+    <collision>
+      <origin xyz="0 0 0.115" rpy="0 0 0"/>
+      <geometry>
+        <cylinder radius="0.03" length="0.21"/>
+      </geometry>
+    </collision>
+  </link>
+  <joint name="camera_joint" type="fixed">
+    <parent link="tool0"/>
+    <child link="camera"/>
+    <origin xyz="0 0 0" rpy="0 0 0"/>
+  </joint>
 </robot>

Commit message: bandaid solution for oblique, will need to improve later

File: src/ur20_sim/urdf/ur20_parked.urdf.xacro (robot description, xacro)
@@ -23,5 +23,14 @@
       <origin xyz="0 0 0.115" rpy="0 0 0"/>
       <geometry>
-        <cylinder radius="0.03" length="0.21"/>
+        <cylinder radius="0.045" length="0.21"/>
+      </geometry>
+    </collision>
+    <!-- Guard volume around the flange area: the UR firmware protective-
+         stops on possible clamping between tool flange and lower arm well
+         before the meshes would touch, so keep planning clear of it. -->
+    <collision>
+      <origin xyz="0 0 0.065" rpy="0 0 0"/>
+      <geometry>
+        <cylinder radius="0.10" length="0.12"/>
       </geometry>
     </collision>
